File: kicad/handipi_kb/handipi_kb.sch (KiCad schematic (older format))
At the start: 87 parts, among them J1 USB_Connector, SW1 SW_Push_Dual, SW10 SW_Push_Dual, SW11 SW_Push_Dual, SW12 SW_Push_Dual, SW13 SW_Push_Dual, SW14 SW_Push_Dual, SW15 SW_Push_Dual, SW16 SW_Push_Dual, SW17 SW_Push_Dual, SW18 SW_Push_Dual, SW19 SW_Push_Dual, SW2 SW_Push_Dual, SW20 SW_Push_Dual, SW21 SW_Push_Dual, SW22 SW_Push_Dual, SW23 SW_Push_Dual, SW24 SW_Push_Dual, SW25 SW_Push_Dual, SW26 SW_Push_Dual, SW27 SW_Push_Dual, SW28 SW_Push_Dual, SW29 SW_Push_Dual, SW3 SW_Push_Dual, SW30 SW_Push_Dual, SW31 SW_Push_Dual, SW32 SW_Push_Dual, SW33 SW_Push_Dual, SW34 SW_Push_Dual, SW35 SW_Push_Dual, SW36 SW_Push_Dual, SW37 RESET, SW38 BOOT, SW39 5-way_switch, SW4 SW_Push_Dual, SW5 SW_Push_Dual, SW6 SW_Push_Dual, SW7 SW_Push_Dual, SW8 SW_Push_Dual, SW9 SW_Push_Dual, U1 ATmega328-PU, Y1 16mhz

Commit message: Clean up structure and V1
Parts:
- removed SW37: RESET, Button_Switch_THT:SW_PUSH_6mm, symbol horizon:SW_Push
- removed SW38: BOOT, Button_Switch_THT:SW_PUSH_6mm, symbol horizon:SW_Push
- added D37, D38: D_Zener, Diode_THT:D_A-405_P7.62mm_Horizontal, symbol Device:D_Zener
- added H1, H2, H3, H4: Hole_Pad, Horizon:Mount_M2, symbol horizon:Hole_Pad
- added J2: RESET, Connector_PinHeader_1.27mm:PinHeader_1x02_P1.27mm_Vertical, symbol Connector:Conn_01x02_Female
- added J3: BOOT, Connector_PinHeader_1.27mm:PinHeader_1x02_P1.27mm_Vertical, symbol Connector:Conn_01x02_Female
- SW1, SW10, SW11, SW12, SW13, SW14, SW15, SW16, SW17, SW18, SW19, SW2, SW20, SW21, SW22, SW23, SW24, SW25, SW26, SW27, SW28, SW29, SW3, SW30, SW31, SW32, SW33, SW34, SW35, SW36, SW4, SW5, SW6, SW7, SW8, SW9: footprint Button_Switch_THT:SW_PUSH_6mm -> RSU:SW_PUSH_6mm_with_hole
Connections:
- net labels added: ROW4
- wire segments 137 -> 146
Other:
- moved on the sheet: R3, R4, SW39
