File: kicad/handipi_kb/handipi_kb.kicad_sch (KiCad schematic)
At the start: 93 parts

Commit message: Fix footprint for directional switch
Parts:
- C1, C2: value (none) -> 22p; footprint (none) -> Capacitor_THT:C_Disc_D3.0mm_W2.0mm_P2.50mm
- C3: value (none) -> 4.7u; footprint (none) -> Capacitor_THT:CP_Radial_D4.0mm_P1.50mm
- C4, C5: value (none) -> 100n; footprint (none) -> Capacitor_THT:C_Disc_D4.3mm_W1.9mm_P5.00mm
- D1, D10, D11, D12, D13, D14, D15, D16, D17, D18, D19, D2, D20, D21, D22, D23, D24, D25, D26, D27, D28, D29, D3, D30, D31, D32, D33, D34, D35, D36, D4, D5, D6, D7, D8, D9: value (none) -> D; footprint (none) -> Diode_SMD:D_SOD-123
- D37, D38: value (none) -> D_Zener; footprint (none) -> Diode_THT:D_A-405_P7.62mm_Horizontal
- H1, H2, H3, H4: value (none) -> Hole_Pad; footprint (none) -> Horizon:Mount_M2
- J1: value (none) -> USB_Connector; footprint (none) -> Connector_PinHeader_1.27mm:PinHeader_1x04_P1.27mm_Vertical
- J2: value (none) -> RESET; footprint (none) -> Connector_PinHeader_1.27mm:PinHeader_1x02_P1.27mm_Vertical
- J3: value (none) -> BOOT; footprint (none) -> Connector_PinHeader_1.27mm:PinHeader_1x02_P1.27mm_Vertical
- R1: value (none) -> 10k; footprint (none) -> Resistor_THT:R_Axial_DIN0207_L6.3mm_D2.5mm_P10.16mm_Horizontal
- R2: value (none) -> 1.5k; footprint (none) -> Resistor_THT:R_Axial_DIN0207_L6.3mm_D2.5mm_P10.16mm_Horizontal
- R3, R4: value (none) -> 75R; footprint (none) -> Resistor_THT:R_Axial_DIN0207_L6.3mm_D2.5mm_P10.16mm_Horizontal
- SW1, SW10, SW11, SW12, SW13, SW14, SW15, SW16, SW17, SW18, SW19, SW2, SW20, SW21, SW22, SW23, SW24, SW25, SW26, SW27, SW28, SW29, SW3, SW30, SW31, SW32, SW33, SW34, SW35, SW36, SW4, SW5, SW6, SW7, SW8, SW9: value (none) -> SW_Push_Dual; footprint (none) -> RSU:SW_PUSH_6mm_with_hole
- SW39: value (none) -> 5-way_switch; footprint (none) -> RSU:switch_5way
- U1: value (none) -> ATmega328-PU; footprint (none) -> Package_DIP:DIP-28_W7.62mm
- Y1: value (none) -> 16mhz; footprint (none) -> Crystal:Crystal_HC18-U_Vertical
Connections:
- net COL6: now also SW39.5 (com); no longer SW39.4 (right)
- net ROW4: now also SW39.4 (right); no longer SW39.5 (com)
